File: space_whistle_pressure.sch (KiCad schematic (older format))
At the start: 15 parts, among them K1 CONN_3, U1 MCP1703, U2 MCP601

Commit message: add Digi-Key part numbers
Parts:
- C1, C2: Digi-Key (none) -> 1276-2872-1-ND
- C3, C6, C7: Digi-Key (none) -> 445-1358-1-ND
- C4, C5: Digi-Key (none) -> 445-1314-1-ND
- C8: Digi-Key (none) -> 1276-1094-1-ND
- R1: Digi-Key (none) -> 311-20.0KHRCT-ND
- RV1: Digi-Key (none) -> TC33X-2-501ECT-ND
- RV2: Digi-Key (none) -> TC33X-2-203ECT-ND
- S1: Digi-Key (none) -> MP3V5010DP-ND
- U1: Digi-Key (none) -> MCP1703T-3302E/CBCT-ND
- U2: Digi-Key (none) -> MCP601T-I/OTCT-ND
Changed lines of the file:
@@
 Sheet 1 1
 Title "Space Whistle Pressure Sensor"
-Date "29 jul 2014"
+Date "4 aug 2014"
 Rev "1"
 Comp "by Open Music Kontrollers (http://open-music-kontrollers.ch)"
@@
 F 2 "~" H 4350 1050 60  0000 C CNN
 F 3 "~" H 4350 1050 60  0000 C CNN
+F 4 "MCP1703T-3302E/CBCT-ND" H 4350 1050 60  0001 C CNN "Digi-Key"
 	1    4350 1050
 	1    0    0    -1
@@
 F 2 "~" H 3988 1050 30  0000 C CNN
 F 3 "~" H 3950 1200 60  0000 C CNN
+F 4 "1276-2872-1-ND" H 3950 1200 60  0001 C CNN "Digi-Key"
 	1    3950 1200
 	1    0    0    -1
@@
 F 2 "~" H 4788 1050 30  0000 C CNN
 F 3 "~" H 4750 1200 60  0000 C CNN
+F 4 "1276-2872-1-ND" H 4750 1200 60  0001 C CNN "Digi-Key"
 	1    4750 1200
 	1    0    0    -1
@@
 F 2 "~" H 2188 750 30  0000 C CNN
 F 3 "~" H 2150 900 60  0000 C CNN
+F 4 "445-1314-1-ND" H 2150 900 60  0001 C CNN "Digi-Key"
 	1    2150 900
 	1    0    0    -1
@@
 F 2 "~" H 3038 1700 30  0000 C CNN
 F 3 "~" H 3000 1850 60  0000 C CNN
+F 4 "445-1314-1-ND" H 3000 1850 60  0001 C CNN "Digi-Key"
 	1    3000 1850
 	1    0    0    -1
@@
 F 2 "~" H 1550 2900 60  0000 C CNN
 F 3 "~" H 1550 2900 60  0000 C CNN
+F 4 "TC33X-2-501ECT-ND" H 1550 2900 60  0001 C CNN "Digi-Key"
 	1    1550 2900
 	1    0    0    -1
@@
 F 2 "~" H 2300 2750 60  0000 C CNN
 F 3 "~" H 2300 2750 60  0000 C CNN
+F 4 "TC33X-2-203ECT-ND" H 2300 2750 60  0001 C CNN "Digi-Key"
 	1    2300 2750
 	1    0    0    -1
@@
 F 2 "~" V 1730 2750 30  0000 C CNN
 F 3 "~" H 1800 2750 30  0000 C CNN
+F 4 "311-20.0KHRCT-ND" V 1800 2750 60  0001 C CNN "Digi-Key"
 	1    1800 2750
 	0    -1   -1   0
@@
 F 2 "~" H 1588 2400 30  0000 C CNN
 F 3 "~" H 1550 2550 60  0000 C CNN
+F 4 "445-1358-1-ND" H 1550 2550 60  0001 C CNN "Digi-Key"
 	1    1550 2550
 	1    0    0    -1
@@
 F 2 "~" H 1988 750 30  0000 C CNN
 F 3 "~" H 1950 900 60  0000 C CNN
+F 4 "445-1358-1-ND" H 1950 900 60  0001 C CNN "Digi-Key"
 	1    1950 900
 	1    0    0    -1
@@
 F 2 "~" H 3238 1700 30  0000 C CNN
 F 3 "~" H 3200 1850 60  0000 C CNN
+F 4 "445-1358-1-ND" H 3200 1850 60  0001 C CNN "Digi-Key"
 	1    3200 1850
 	1    0    0    -1
@@
 F 2 "" H 3100 2450 60  0000 C CNN
 F 3 "" H 3100 2450 60  0000 C CNN
+F 4 "MCP601T-I/OTCT-ND" H 3100 2450 60  0001 C CNN "Digi-Key"
 	1    3100 2450
 	1    0    0    -1
@@
 F 2 "MODULE" H 2900 1200 50  0001 C CNN
 F 3 "DOCUMENTATION" H 2900 1200 50  0001 C CNN
+F 4 "MP3V5010DP-ND" H 2900 1200 60  0001 C CNN "Digi-Key"
 	1    2900 1200
 	1    0    0    -1
@@
 F 2 "~" H 2188 1350 30  0000 C CNN
 F 3 "~" H 2150 1500 60  0000 C CNN
+F 4 "1276-1094-1-ND" H 2150 1500 60  0001 C CNN "Digi-Key"
 	1    2150 1500
 	1    0    0    -1
